File: chipysat.kicad_sch (KiCad schematic)
At the start: 291 parts, among them J1 FTS-105-01-X-DV-A, J10 TFM-110-12-X-D-A, J11 USB_C_Receptacle_USB2.0, J12 02x05 M 1.27mm, J13 Conn_01x08, J14 Conn_01x08, J15 TFM-110-12-X-D-A, J16 FLE-107-01-X-DV-A, J17 USD-1040310811, J18 MOLEX_5051102491, J6 Micro_SD_Card, J7 U.FL-R-SMT-1, J8 USB_C_Receptacle_USB2.0, J9 SFC-110-T2-X-D-A, Q1 NX3008NBKS, Q10 NX3008NBKS, Q11 MBT2222ADW1T1, Q12 MBT2222ADW1T1, Q13 NX3008NBKS, Q14 NX3008NBKS, Q15 MBT2222ADW1T1, Q16 MBT2222ADW1T1, Q17 MMBT2907, Q18 MMBT2907, Q19 IRLML2803, Q2 NX3008NBKS, Q20 SQ3495EV-T1, Q21 SQ3495EV-T1, Q3 MBT2222ADW1T1, Q4 MBT2222ADW1T1, Q5 NX3008NBKS, Q6 NX3008NBKS, Q7 MBT2222ADW1T1, Q8 MBT2222ADW1T1, Q9 NX3008NBKS, SW2 CAS-120TA, SW3 KMR2x, SW4 CAS-120TA, U1 MAX706RESA+, U10 RFM98PW, U11 BNO085, U12 USBLC6-2SC6, U13 STM32H743VITx, U14 WE-TVS-82400102, U15 LTC4412xS6, U16 XC6210B332MR-G, U17 AP7366-28W5-7, U18 TLV75515PDBVR, U19 BQ25570RGRR, U2 DRV8830DRC, U20 MAX40200AUK, U3 OPT4001, U4 LTC4412xS6, U5 DRV8830DRC, U6 PCF8523TK, U7 DRV8830DRC, U8 AP2112K-3.3, U9 MR25H40, Y2 32.768kHz/7pF, Y3 32.768kHz/12.5pF, Y4 12MHz/7pF

Commit message: Add a few solar cells
Parts:
- removed C1, C13, C2, C3, C4, C5, C6, C7, C8: 10nF, Capacitor_SMD:C_0603_1608Metric, symbol Device:C
- removed C10: 0.1uF, Capacitor_SMD:C_0402_1005Metric, symbol Device:C
- removed C11, C21, C23, C24: 0.1uF, Capacitor_SMD:C_0603_1608Metric, symbol Device:C
- removed C12, C18: 4.7uF, Capacitor_SMD:C_0603_1608Metric, symbol Device:C
- removed C14, C20, C27, C30, C33, C35, C36, C40, C41, C46, C48, C49, C50, C55, C9: 0.1uF, Capacitor_SMD:C_0603_1608Metric, symbol Device:C_Small
- removed C15: 1uF, Capacitor_SMD:C_0603_1608Metric, symbol Device:C
- removed C16: 100uF, Capacitor_SMD:C_0805_2012Metric, symbol Device:C
- removed C17, C22, C28, C52, C53, C54, C56, C60, C61, C62, C63, C64, C66: 1uF, Capacitor_SMD:C_0603_1608Metric, symbol Device:C_Small
- removed C19: 22uF, Capacitor_SMD:C_0603_1608Metric, symbol Device:C
- removed C25, C26, C57, C58, C59, C68, C72: 10uF, Capacitor_SMD:C_0603_1608Metric, symbol Device:C_Small
- removed C29, C31: 10uF, Capacitor_SMD:C_0805_2012Metric, symbol Device:C_Small
- removed C32: 1uF, Capacitor_SMD:C_0805_2012Metric, symbol Device:C_Small
- removed C34, C42: 4.7nF, Capacitor_SMD:C_0603_1608Metric, symbol Device:C_Small
- removed C37, C38: 22pF, Capacitor_SMD:C_0603_1608Metric, symbol Device:C_Small
- removed C39, C67: 47uF, Capacitor_Tantalum_SMD:CP_EIA-2012-12_Kemet-R, symbol Device:C_Polarized_Small_US
- removed C43, C47: 2.2uF, Capacitor_SMD:C_0603_1608Metric, symbol Device:C_Small
- removed C44, C45: 4pF, Capacitor_SMD:C_0603_1608Metric, symbol Device:C_Small
- removed C51: 10nF, Capacitor_SMD:C_0603_1608Metric, symbol Device:C_Small
- removed D1, D3: MBR1020VL-AU_R1, Diode_SMD:D_SOD-123F, symbol Device:D_Schottky_Small
- removed D5, D6, D7: DFLS130L-7, Diode_SMD:D_PowerDI-123, symbol Device:D_Schottky
- removed FB1: 120R, Inductor_SMD:L_0603_1608Metric, symbol Device:FerriteBead_Small
- removed FL1, FL2, FL3: SRF2012, mainboard:SRF2012, symbol Device:Filter_EMI_CommonMode
- removed H1, H2, H3, H4, H5, H6, H7, H8: MountingHole_Pad, mainboard:MountingHole, symbol Mechanical:MountingHole_Pad
- removed J1: FTS-105-01-X-DV-A, solarpanels:SAMTEC-FTS-105-01-X-DV-A, symbol Connector_Generic:Conn_02x05_Odd_Even
- removed J10, J15: TFM-110-12-X-D-A, mainboard:SAMTEC_TFM-110-12-X-D-A, symbol Connector_Generic:Conn_02x10_Odd_Even
- removed J11, J8: USB_C_Receptacle_USB2.0, Connector_USB:USB_C_Receptacle_HRO_TYPE-C-31-M-12, symbol Connector:USB_C_Receptacle_USB2.0
- removed J12: 02x05 M 1.27mm, Connector_PinHeader_1.27mm:PinHeader_2x05_P1.27mm_Vertical_SMD, symbol Connector_Generic:Conn_02x05_Odd_Even
- removed J13, J14: Conn_01x08, Connector_PinHeader_2.54mm:PinHeader_1x08_P2.54mm_Vertical, symbol Connector_Generic:Conn_01x08
- removed J16: FLE-107-01-X-DV-A, cameraboard:SAMTEC_FLE-107-01-X-DV-A, symbol Connector_Generic:Conn_02x07_Odd_Even
- removed J17: USD-1040310811, Connector_Card:microSD_HC_Molex_104031-0811, symbol cameraboard:USD-1040310811
- removed J18: MOLEX_5051102491, cameraboard:MOLEX_5051102491, symbol cameraboard:MOLEX_5051102491
- removed J6: Micro_SD_Card, mainboard:microSD_104031-0811, symbol Connector:Micro_SD_Card_Det2
- removed J7: U.FL-R-SMT-1, mainboard:U.FL-R-SMT-1, symbol mainboard:U.FL-R-SMT-1
- removed J9: SFC-110-T2-X-D-A, mainboard:SAMTEC_SFC-110-T2-X-D-A, symbol Connector_Generic:Conn_02x10_Odd_Even
- removed Q1, Q10, Q13, Q14, Q2, Q5, Q6, Q9: NX3008NBKS, Package_TO_SOT_SMD:SOT-363_SC-70-6, symbol mainboard:NX3008NBKS
- removed Q11, Q12, Q15, Q16, Q3, Q4, Q7, Q8: MBT2222ADW1T1, Package_TO_SOT_SMD:SOT-363_SC-70-6, symbol Transistor_BJT:MBT2222ADW1T1
- removed Q17, Q18: MMBT2907, Package_TO_SOT_SMD:SOT-23, symbol mainboard:MMBT2907
- removed Q19: IRLML2803, Package_TO_SOT_SMD:SOT-23, symbol Transistor_FET:IRLML2060
- removed Q20, Q21: SQ3495EV-T1, Package_TO_SOT_SMD:SOT-23-6, symbol cameraboard:SQ3495EV-T1
- removed R1, R11, R12, R2, R21, R22, R39, R40: 680R, Resistor_SMD:R_0603_1608Metric, symbol Device:R_US
- removed R10, R18, R20, R36, R38, R48, R50, R68, R8: 200K, Resistor_SMD:R_0603_1608Metric, symbol Device:R_US
- removed R100, R101, R103, R104, R106, R107, R108, R109, R110, R111, R112, R96: 10K, Resistor_SMD:R_0603_1608Metric, symbol Device:R_Small
- removed R102: 100R, Resistor_SMD:R_0603_1608Metric, symbol Device:R_Small
- removed R105: 1K, Resistor_SMD:R_0603_1608Metric, symbol Device:R_Small
- removed R113, R114, R115, R116, R118, R72, R73: 0R, Resistor_SMD:R_0603_1608Metric, symbol Device:R_Small_US
- removed R117, R76: DNI (0R), Resistor_SMD:R_0603_1608Metric, symbol Device:R_Small_US
- removed R13, R14, R23, R24, R3, R4, R41, R42, R90: 100K, Resistor_SMD:R_0603_1608Metric, symbol Device:R_US
- removed R15, R16, R17, R19, R33, R34, R35, R37, R45, R46, R47, R49, R5, R6, R7, R77, R78, R79, R80, R81, R84, R88, R9: 10K, Resistor_SMD:R_0603_1608Metric, symbol Device:R_US
- removed R25, R26, R27, R28, R29, R30, R31, R32, R43, R44, R61: DNI (0R), Resistor_SMD:R_0603_1608Metric, symbol Device:R_US
- removed R51, R52, R60, R69, R74, R82, R89, R91, R92, R93: 0R, Resistor_SMD:R_0603_1608Metric, symbol Device:R_US
- removed R53, R54: 4.7K, Resistor_SMD:R_0603_1608Metric, symbol Device:R_US
- removed R55, R56, R57, R58, R75: 1K, Resistor_SMD:R_0603_1608Metric, symbol Device:R_US
- removed R59, R62: 0R, Resistor_SMD:R_0402_1005Metric, symbol Device:R_Small_US
- removed R63: 7.32M, Resistor_SMD:R_0603_1608Metric, symbol Device:R_Small_US
- removed R64: 5.62M, Resistor_SMD:R_0603_1608Metric, symbol Device:R_Small_US
- removed R65: 374K, Resistor_SMD:R_0603_1608Metric, symbol Device:R_Small_US
- removed R66, R70: 8.25M, Resistor_SMD:R_0603_1608Metric, symbol Device:R_Small_US
- removed R67: 4.53M, Resistor_SMD:R_0603_1608Metric, symbol Device:R_Small_US
- removed R71: 4.75M, Resistor_SMD:R_0603_1608Metric, symbol Device:R_Small_US
- removed R83: 1M, Resistor_SMD:R_0603_1608Metric, symbol Device:R_US
- removed R85, R86: 5.1K, Resistor_SMD:R_0603_1608Metric, symbol Device:R_US
- removed R87, R94: 22R, Resistor_SMD:R_0603_1608Metric, symbol Device:R_US
- removed R95: 1M, Resistor_SMD:R_0603_1608Metric, symbol Device:R_Small
- removed R97: 0R, Resistor_SMD:R_0603_1608Metric, symbol Device:R_Small
- removed R98, R99: 5.1K, Resistor_SMD:R_0603_1608Metric, symbol Device:R_Small
- removed SC1, SC2, SC3, SC4, SC5, SC6, SC7, SC8: SolarCell_Small, solarpanels:KXOB25-05X3F, symbol solarpanels:SolarCell_Small
- removed SW2, SW4: CAS-120TA, cameraboard:CAS-120TA, symbol Switch:SW_SPDT
- removed SW3: KMR2x, mainboard:BTN_KMR2, symbol Switch:SW_Push
- removed TP1, TP2, TP3, TP4: TP, TestPoint:TestPoint_THTPad_D1.0mm_Drill0.5mm, symbol Connector:TestPoint
- removed U1: MAX706RESA+, Package_SO:SOIC-8_3.9x4.9mm_P1.27mm, symbol mainboard:MAX708RESA+
- removed U10: RFM98PW, mainboard:RFM98PW, symbol mainboard:RFM98PW
- removed U11: BNO085, mainboard:BNO085, symbol mainboard:BNO085
- removed U12: USBLC6-2SC6, Package_TO_SOT_SMD:SOT-23-6, symbol Power_Protection:USBLC6-2SC6
- removed U13: STM32H743VITx, Package_QFP:LQFP-100_14x14mm_P0.5mm, symbol MCU_ST_STM32H7:STM32H743VITx
- removed U14: WE-TVS-82400102, Package_TO_SOT_SMD:SOT-23-6, symbol Power_Protection:USBLC6-2SC6
- removed U15, U4: LTC4412xS6, Package_TO_SOT_SMD:TSOT-23-6, symbol Power_Management:LTC4412xS6
- removed U16: XC6210B332MR-G, Package_TO_SOT_SMD:SOT-23-5, symbol Regulator_Linear:AP2127K-2.8
- removed U17: AP7366-28W5-7, Package_TO_SOT_SMD:SOT-23-5, symbol Regulator_Linear:AP2127K-2.8
- removed U18: TLV75515PDBVR, Package_TO_SOT_SMD:SOT-23-5, symbol Regulator_Linear:AP2127K-2.8
- removed U19: BQ25570RGRR, solarpanels:QFN50P350X350X100-21N-D, symbol solarpanels:BQ25570RGRR
- removed U2, U5, U7: DRV8830DRC, mainboard:VSON-10, symbol mainboard:DRV8830DRC
- removed U3: OPT4001, Package_TO_SOT_SMD:SOT-583-8, symbol solarpanels:OPT4001
- removed U6: PCF8523TK, Package_SON:HVSON-8-1EP_4x4mm_P0.8mm_EP2.2x3.1mm, symbol Timer_RTC:PCF8523TK
- removed U8: AP2112K-3.3, Package_TO_SOT_SMD:SOT-23-5, symbol Regulator_Linear:AP2112K-3.3
- removed U9: MR25H40, mainboard:MR25H40DF, symbol Memory_NVRAM:MR25H40
- removed Y2: 32.768kHz/7pF, Crystal:Crystal_SMD_MicroCrystal_CC7V-T1A-2Pin_3.2x1.5mm, symbol Device:Crystal_Small
- removed Y3: 32.768kHz/12.5pF, Crystal:Crystal_SMD_MicroCrystal_CC7V-T1A-2Pin_3.2x1.5mm, symbol Device:Crystal_Small
- removed Y4: 12MHz/7pF, Crystal:Crystal_SMD_2520-4Pin_2.5x2.0mm, symbol Device:Crystal_GND24_Small
- added C45, C63, C64, C72: 0.1uF, Capacitor_SMD:C_0603_1608Metric, symbol Device:C
- added C46, C61: 4.7uF, Capacitor_SMD:C_0603_1608Metric, symbol Device:C
- added C48: 10nF, Capacitor_SMD:C_0603_1608Metric, symbol Device:C
- added C56: 1uF, Capacitor_SMD:C_0603_1608Metric, symbol Device:C
- added C57: 100uF, Capacitor_SMD:C_0805_2012Metric, symbol Device:C
- added C62: 22uF, Capacitor_SMD:C_0603_1608Metric, symbol Device:C
- added C67: 10uF, Capacitor_SMD:C_0603_1608Metric, symbol Device:C_Small
- added D8, D9: DFLS130L-7, Diode_SMD:D_PowerDI-123, symbol Device:D_Schottky
- added J13: MOLEX_5051102491, cameraboard:MOLEX_5051102491, symbol cameraboard:MOLEX_5051102491
- added R100, R98: 8.25M, Resistor_SMD:R_0603_1608Metric, symbol Device:R_Small_US
- added R101: 4.75M, Resistor_SMD:R_0603_1608Metric, symbol Device:R_Small_US
- added R106, R111: DNI (0R), Resistor_SMD:R_0603_1608Metric, symbol Device:R_Small_US
- added R109, R110, R112: 0R, Resistor_SMD:R_0603_1608Metric, symbol Device:R_Small_US
- added R93: 7.32M, Resistor_SMD:R_0603_1608Metric, symbol Device:R_Small_US
- added R94: 5.62M, Resistor_SMD:R_0603_1608Metric, symbol Device:R_Small_US
- added R97: 374K, Resistor_SMD:R_0603_1608Metric, symbol Device:R_Small_US
- added R99: 4.53M, Resistor_SMD:R_0603_1608Metric, symbol Device:R_Small_US
- added SC10, SC11, SC9: SolarCell, solarpanels:KXOB25-05X3F, symbol solarpanels:SolarCell_Small
- added U16: BQ25570RGRR, solarpanels:QFN50P350X350X100-21N-D, symbol solarpanels:BQ25570RGRR
- added U21: STM32U595VJTxQ, Package_QFP:LQFP-100_14x14mm_P0.5mm, symbol MCU_ST_STM32U5:STM32U595VJTxQ
- C69: value 1uF -> 0.1uF
- C70: value 0.1uF -> 1uF
- C71: value 1uF -> 10uF
Connections:
- net +3.3V: no longer C69.2
- net +3V3: now also C72.1
- net 1.5V: now also C70.1, J13.15 (Pin_15); no longer C65.1
- net 2.8V: now also C65.1, C67.1, J13.14 (Pin_14)
- net BATT_P: now also R112.1
- net DCMI_CLK: now also J13.12 (Pin_12)
- net DCMI_D0: now also J13.6 (Pin_6)
- net DCMI_D1: now also J13.4 (Pin_4)
- net DCMI_D2: now also J13.3 (Pin_3)
- net DCMI_D3: now also J13.5 (Pin_5)
- net DCMI_D4: now also J13.7 (Pin_7)
- net DCMI_D5: now also J13.9 (Pin_9)
- net DCMI_D6: now also J13.11 (Pin_11)
- net DCMI_D7: now also J13.13 (Pin_13)
- net DCMI_HSYNC: now also J13.16 (Pin_16)
- net DCMI_PCLK: now also J13.8 (Pin_8)
- net DCMI_PWDN: now also J13.17 (Pin_17)
- net DCMI_RST: now also J13.19 (Pin_19)
- net DCMI_VSYNC: now also J13.18 (Pin_18)
- net GND: now also C69.2, C45.2, C46.2, C48.2, C56.2, C57.2, C61.2, C62.2, C63.2, C64.2, C67.2, C72.2, J13.10 (Pin_10), J13.23 (Pin_23), J13.P1, J13.P2, R101.1, R111.1, R94.1, R99.1, U16.1 (VSS_2), U16.15 (VSS), U16.17 (NC), U16.21 (PAD), U16.5 (EN_N), U16.9 (NC_2); no longer C69.1
- net I2C1_SCL: now also J13.20 (Pin_20)
- net I2C1_SDA: now also J13.22 (Pin_22)
- net VBAT: now also C57.1, R112.2, U16.18 (VBAT)
- net VBAT_OK: now also R110.1, U16.13 (VBAT_OK)
- net VOUT_EN: now also C56.1, R110.2, U16.6 (VOUT_EN)
- net VSOLAR: now also C45.1, C46.1, D9.1 (K), R106.2, U16.2 (VIN_DC)
- net at FB2.2: now also C69.1, J13.21 (Pin_21); no longer C70.1
- net at L2.2, U20.1 (VDD), U20.3 (EN): now also C62.1, C64.1, U16.14 (VOUT)
- net at L1.2: now also U16.20 (LBOOST)
- net at L2.1: now also U16.16 (LBUCK)
- new net: R100.1, R101.2, U16.12 (VOUT_SET)
- new net: R97.1, R98.2, U16.10 (OK_HYST)
- new net: R100.2, R93.2, R97.2, U16.8 (VRDIV)
- new net: R93.1, R94.2, U16.7 (VBAT_OV)
- new net: R98.1, R99.2, U16.11 (OK_PROG)
- new net: D8.1 (K), D9.2 (A), SC10.1 (V+), SC11.1 (V+), SC9.1 (V+)
- new net: D8.2 (A), SC10.2 (V-), SC11.2 (V-), SC9.2 (V-)
- new net: C61.1, C63.1, R109.1, U16.19 (VSTOR)
- new net: R106.1, R109.2, R111.2, U16.3 (VOC_SAMP)
- new net: C48.1, U16.4 (VREF_SAMP)
- new net: U21.10 (VSS), U21.26 (VSS), U21.50 (VSS), U21.74 (VSS), U21.99 (VSS)
- no-connect marks 59 -> 3
Other:
- added sheet Old Stuff (old_stuff.kicad_sch)
- note added: "MCU (STM32U595VJT3Q)"
- note removed: "(Not Populated)"
- note removed: "->"
- note removed: "0x68"
- note removed: "<-"
- note removed: "Arrows indicate clockwise (while facing layer 1)"
- note removed: "Bus Protection - Bypass Jumpers"
- note removed: "COIL+"
- note removed: "COIL-"
- note removed: "Check Xtal Datasheet This value assumes 7pF crystal bulk capacitance"
- note removed: "Coil"
- note removed: "Coil Driver Circuits"
- note removed: "Current Limiting Resistor < 1 Ohm"
- note removed: "Default HI_POW to USB power. Use battery power when USB absent."
- note removed: "ESR < 100 mOhm Tol < 20%"
- note removed: "FLASH STORAGE"
- note removed: "From Top Batteryboard"
- note removed: "Grounded Mounting Holes"
- note removed: "HI-POW SELECT"
- note removed: "HI-Power Selection"
- note removed: "High Power Line Source Selection"
- note removed: "I2C Bus Protection - Motor1"
- note removed: "I2C Bus Protection - Motor2"
- note removed: "I2C Bus Protection - Motor3"
- note removed: "I2C Bus Protection - RTC"
- note removed: "I2C1 ADDR"
- note removed: "IMU"
- note removed: "IMU datasheet recommends 12.5pF crystal capacitance"
- note removed: "LDOs"
- note removed: "Light Sensor"
- note removed: "MCU (STM32H743VITx)"
- note removed: "Motor 1 Jumpers"
- note removed: "Motor 2 Jumpers"
- note removed: "Motor 3 Jumpers"
- note removed: "Mounting Holes"
- note removed: "NOTE"
- note removed: "Only one resistor per side (COIL_P/COIL_N) should be populated. R12 and R18 should nominally be correct."
- note removed: "Potentially Replace with Ferrite Bead"
- note removed: "Power Capacitors (0805)"
- note removed: "Power Enable Circuit"
- note removed: "REAL TIME CLOCK"
- note removed: "REGULATOR"
- note removed: "RTC Jumpers"
- note removed: "RTC supports 7pF (default) and 12.5pF crystal capacitance only"
- note removed: "Radio Jumper"
- note removed: "Reset & Boot0 Switches"
- note removed: "SD Card"
- note removed: "SD Card Connector"
- note removed: "SD Card Jumper"
- note removed: "SPI Bus Protection - Radio"
- note removed: "SPI Bus Protection - SD Card"
- note removed: "STACK CONN"
- note removed: "SWD Connector"
- note removed: "Select boot mode Set "low" for normal operation. Set "high" for bootloader mode"
- note removed: "Set for flight"
- note removed: "Shield"
- note removed: "Solar Cells"
- note removed: "Solar Panel Board +Y"
- note removed: "Stack Connector"
- note removed: "Stack Connectors"
- note removed: "Status LED & IO headers"
- note removed: "TO BOTTOM BATTERYBOARD"
- note removed: "TO PAYLOADBOARD"
- note removed: "TORQUER DRIVERS"
- note removed: "Test Points"
- note removed: "These novel bus protection circuits prevent traditional I2C/SPI failure modes where a single slave failure can disable the entire bus. Learn more: https://doi.org/10.36227/techrxiv.15166620 By default, slave clock and/or data lines can be held low and the Master (SAMD51) will still be able to communicate with the remainder of the bus. They can individually be bypassed by removing the transistor(s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"
- note removed: "To -Y Board"
- note removed: "To Mainboard"
- note removed: "Toggle LDO power on or controlled by Mainboard enable line (defaults to power off)"
- note removed: "UHF RADIO"
- note removed: "USB CONN"
- note removed: "USB Connector"
- note removed: "USB ESD Protection"
- note removed: "WATCH-DOG TIMER"
- note removed: "WDT able to reset MCU when WDT_EN is high"
- note removed: "X BOARD COILS I2C1 ADDR 0x60"
- note removed: "Y BOARD COILS I2C1 ADDR 0x61"
- note removed: "Z BOARD COILS I2C1 ADDR 0x64"
- note removed: "cameraboard"
- note removed: "mainboard"

Commit message: Complete MCU planning
Parts:
- removed SC10, SC11: SolarCell, solarpanels:KXOB25-05X3F, symbol solarpanels:SolarCell_Small
- added C100: 100uF, Capacitor_SMD:C_0603_1608Metric, symbol Device:C_Small
- added C101: 1uF, Capacitor_SMD:C_0603_1608Metric, symbol Device:C_Small
- added C14: 0.1uF, Capacitor_SMD:C_0402_1005Metric, symbol Device:C
- added C2, C89, C90, C93, C94, C95, C96, C97: 0.1uF, Capacitor_SMD:C_0603_1608Metric, symbol Device:C_Small
- added C75, C82, C83, C84: 0.1uF, Capacitor_SMD:C_0603_1608Metric, symbol Device:C
- added C76, C80: 4.7uF, Capacitor_SMD:C_0603_1608Metric, symbol Device:C
- added C77: 10nF, Capacitor_SMD:C_0603_1608Metric, symbol Device:C
- added C78: 1uF, Capacitor_SMD:C_0603_1608Metric, symbol Device:C
- added C79: 100uF, Capacitor_SMD:C_0805_2012Metric, symbol Device:C
- added C81: 22uF, Capacitor_SMD:C_0603_1608Metric, symbol Device:C
- added C85, C86, C87, C88: 4pF, Capacitor_SMD:C_0603_1608Metric, symbol Device:C_Small
- added C91, C92: 2.2uF, Capacitor_SMD:C_0603_1608Metric, symbol Device:C_Small
- added C98, C99: 10uF, Capacitor_SMD:C_0603_1608Metric, symbol Device:C_Small
- added D10, D11, D12, D13, D5, D6: DFLS130L-7, Diode_SMD:D_PowerDI-123, symbol Device:D_Schottky
- added D14, D15: LTST-C190AKT, LED_SMD:LED_0603_1608Metric, symbol Device:LED_Small
- added D7: SZMM5Z5V1T1G, Diode_SMD:D_SOD-523, symbol Diode:Z1SMAxxx
- added H13, H14, H15, H16: MountingHole, solarpanels:MountingHole_2.2mm_M2_DIN965_Pad_TopBottom, symbol Mechanical:MountingHole_Pad
- added L3: 22uH-LPS4018-223MR, solarpanels:LPS4018, symbol Device:L
- added L4: 10uH-LPS4018-103MR, solarpanels:LPS4018, symbol Device:L
- added L5: 2.2uH, symbol Device:L_Small
- added Q1: IRLML2803, Package_TO_SOT_SMD:SOT-23, symbol Transistor_FET:IRLML2060
- added R1: 0R, Resistor_SMD:R_0603_1608Metric, symbol Device:R_US
- added R120: 7.32M, Resistor_SMD:R_0603_1608Metric, symbol Device:R_Small_US
- added R121: 5.62M, Resistor_SMD:R_0603_1608Metric, symbol Device:R_Small_US
- added R122: 374K, Resistor_SMD:R_0603_1608Metric, symbol Device:R_Small_US
- added R123, R125: 8.25M, Resistor_SMD:R_0603_1608Metric, symbol Device:R_Small_US
- added R124: 4.53M, Resistor_SMD:R_0603_1608Metric, symbol Device:R_Small_US
- added R126: 4.75M, Resistor_SMD:R_0603_1608Metric, symbol Device:R_Small_US
- added R127, R129, R130, R133: DNI (0R), Resistor_SMD:R_0603_1608Metric, symbol Device:R_Small_US
- added R128, R131, R132: 0R, Resistor_SMD:R_0603_1608Metric, symbol Device:R_Small_US
- added R13, R14: 0R, Resistor_SMD:R_0402_1005Metric, symbol Device:R_Small_US
- added R134, R135: 1M, Resistor_SMD:R_0603_1608Metric, symbol Device:R_Small_US
- added R136: 16k, Resistor_SMD:R_0603_1608Metric, symbol Device:R_Small_US
- added R137: 33k, Resistor_SMD:R_0603_1608Metric, symbol Device:R_Small_US
- added R139: 240k, Resistor_SMD:R_0603_1608Metric, symbol Device:R_Small_US
- added R140: 680k, Resistor_SMD:R_0603_1608Metric, symbol Device:R_Small_US
- added R2: DNI (0R), Resistor_SMD:R_0603_1608Metric, symbol Device:R_US
- added R3: 200K, Resistor_SMD:R_0603_1608Metric, symbol Device:R_US
- added SC1, SC2, SC3, SC4, SC5: SolarCell, solarpanels:KXOB25-05X3F, symbol solarpanels:SolarCell_Small
- added U1: MAX706RESA+, Package_SO:SOIC-8_3.9x4.9mm_P1.27mm, symbol mainboard:MAX708RESA+
- added U12: OPT4001, Package_TO_SOT_SMD:SOT-583-8, symbol solarpanels:OPT4001
- added U23: BQ25570RGRR, solarpanels:QFN50P350X350X100-21N-D, symbol solarpanels:BQ25570RGRR
- added U24: MAX40200AUK, Package_TO_SOT_SMD:SOT-23-5, symbol Analog_Switch:MAX40200AUK
- added Y4: 12MHz/7pF, Crystal:Crystal_SMD_2520-4Pin_2.5x2.0mm, symbol Device:Crystal_GND24_Small
- added Y5: 32.768kHz/7pF, Crystal:Crystal_SMD_MicroCrystal_CC7V-T1A-2Pin_3.2x1.5mm, symbol Device:Crystal_Small
Connections:
- net +3.3V: now also D14.1 (K)
- net +3V3: now also U21.100 (VDD), U21.11 (VDD), U21.27 (VDD), U21.51 (VDD), U21.73 (VDDUSB), U21.75 (VDD), C14.1, C2.1, C89.1, C90.1, C93.1, C94.1, C95.1, C96.1, C97.1, C98.1, R13.1, R132.1, R133.1, U1.2 (VCC), U12.1 (VDD); no longer C72.1, U20.5 (OUT)
- net BATT_P: now also R131.1
- net DCMI_D0: now also U21.66 (PC9)
- net DCMI_D1: now also U21.65 (PC8)
- net DCMI_D2: now also U21.64 (PC7)
- net DCMI_D3: now also U21.63 (PC6)
- net DCMI_D4: now also U21.3 (PE4)
- net DCMI_D5: now also U21.84 (PD3)
- net DCMI_D6: now also U21.4 (PE5)
- net DCMI_D7: now also U21.5 (PE6)
- net DCMI_HSYNC: now also U21.28 (PA4)
- net DCMI_VSYNC: now also U21.93 (PB7)
- net GND: now also D8.2 (A), SC9.2 (V-), U21.10 (VSS), U21.19 (VSSA), U21.26 (VSS), U21.48 (VSSSMPS), U21.50 (VSS), U21.74 (VSS), U21.99 (VSS), C100.2, C101.2, C14.2, C2.2, C75.2, C76.2, C77.2, C78.2, C79.2, C80.2, C81.2, C82.2, C83.2, C84.2, C85.1, C86.2, C87.1, C88.1, C89.2, C90.2, C91.2, C92.2, C93.2, C94.2, C95.2, C96.2, C97.2, C98.2, C99.2, D10.2 (A), D7.2 (A), H13.1, H14.1, H15.1, H16.1, R121.1, R124.1, R126.1, R130.1, R134.2, R135.2, R136.2, R137.2, R14.2, R140.1, R3.2, SC3.2 (V-), U1.3 (GND), U1.4 (PFI), U12.4 (GND), U23.1 (VSS_2), U23.15 (VSS), U23.17 (NC), U23.21 (PAD), U23.5 (EN_N), U23.9 (NC_2), U24.2 (GND), Y4.2, Y4.4
- net LED_B: now also U21.37 (PE9)
- net LED_G: now also U21.36 (PE8)
- net LED_R: now also U21.35 (PE7)
- net VBAT: now also C79.1, R131.2, U23.18 (VBAT)
- net VBAT_OK: now also U21.16 (PC1); no longer R110.1, U16.13 (VBAT_OK)
- net at D8.1 (K), SC9.1 (V+): now also D5.2 (A), SC1.2 (V-); no longer D9.2 (A)
- net WDT_WDI: now reaches U21.1 (PE2)
- net WDT_WDI: now also U1.6 (~{WDI})
- net XTAL_IN: now reaches U21.13 (PH1)
- net XTAL_IN: now also C85.2, Y4.3
- net ~{RESET}: now reaches U21.14 (NRST)
- net ~{RESET}: now also Q1.3 (D), R2.1
- net LPUART_RX: now reaches U21.15 (PC0)
- net WDT_EN: now reaches U21.2 (PE3)
- net WDT_EN: now also Q1.1 (G), R3.1
- net VDDA: now reaches U21.20 (VREF+)
- net VDDA: now also U21.21 (VDDA), C100.1, C101.1
- net SDMMC_CMD: now reaches U21.22 (PA0)
- net LPUART_TX: now reaches U21.24 (PA2)
- net SPI_RF_SCK: now reaches U21.29 (PA5)
- net DCMI_PIXCLK: now reaches U21.30 (PA6)
- net HEATER0: now reaches U21.31 (PA7)
- net SPI_RF_NSS: now reaches U21.32 (PB0)
- net HEATER1: now reaches U21.33 (PB1)
- net RF_IO1: now reaches U21.39 (PE11)
- net RF_IO0: now reaches U21.40 (PE12)
- net RF_RST: now reaches U21.41 (PE13)
- net SPI_RF_MISO: now reaches U21.42 (PE14)
- net SPI_RF_MOSI: now reaches U21.43 (PE15)
- net I2C_LIGHT_SCL: now reaches U21.44 (PB10)
- net I2C_LIGHT_SCL: now also U12.5 (SCL)
- net I2C_LIGHT_SCA: now reaches U21.45 (PB11)
- net at U21.46 (VLXSMPS): now also L5.2
- net VDDSMPS: now reaches U21.47 (VDDSMPS)
- net VDDSMPS: now also C99.1
- net VDD11: now reaches U21.49 (VDD11)
- net VDD11: now also U21.98 (VDD11), C91.1, C92.1
- net SDMMC_D0: now reaches U21.53 (PB14)
- net SDMMC_D1: now reaches U21.54 (PB15)
- net USART_IMU_TX: now reaches U21.55 (PD8)
- net USART_IMU_RX: now reaches U21.56 (PD9)
- net IMU_INT: now reaches U21.57 (PD10)
- net IMU_RST: now reaches U21.58 (PD11)
- net at U21.6 (VBAT): now also R139.1, R140.2
- net CAM_RST: now reaches U21.61 (PD14)
- net CAM_CLK: now reaches U21.62 (PD15)
- net BURN0: now reaches U21.67 (PA8)
- net BURN1: now reaches U21.68 (PA9)
- net USB_D-: now reaches U21.70 (PA11)
- net USB_D+: now reaches U21.71 (PA12)
- net DBG_SWDIO: now reaches U21.72 (PA13)
- net DBG_SWCLK: now reaches U21.76 (PA14)
- net SPI_FLASH_NSS: now reaches U21.77 (PA15)
- net SPI_FLASH_SCK: now reaches U21.78 (PC10)
- net SPI_FLASH_MISO: now reaches U21.79 (PC11)
- net at U21.8 (PC14): now also C87.2, Y5.2
- net SPI_FLASH_MOSI: now reaches U21.80 (PC12)
- net FLASH_IO2: now reaches U21.81 (PD0)
- net FLASH_IO3: now reaches U21.82 (PD1)
- net SDMMC_CK: now reaches U21.87 (PD6)
- net SDMMC_D2: now reaches U21.89 (PB3)
- net at U21.9 (PC15): now also C88.2, Y5.1
- net SDMMC_D3: now reaches U21.90 (PB4)
- net SD_CD: now reaches U21.91 (PB5)
- net I2C_CURR_SCL: now reaches U21.92 (PB6)
- net XTAL_OUT: now reaches U21.94 (PH3)
- net XTAL_OUT: now also C86.1, Y4.1
- net I2C_CURR_SDA: now reaches U21.96 (PB9)
- net VOUT_EN renamed VOUT_EN_TOP
- net VOUT_EN_TOP: now also R134.1
- net VSOLAR renamed VSOLAR_TOP
- new net: C72.1, R132.2, U20.5 (OUT)
- new net: R13.2, R14.1, U12.2 (ADDR)
- new net: R125.1, R126.2, U23.12 (VOUT_SET)
- new net: R120.1, R121.2, U23.7 (VBAT_OV)
- new net: D5.1 (K), D6.2 (A), SC1.1 (V+), SC2.2 (V-)
- new net: R120.2, R122.2, R125.2, U23.8 (VRDIV)
- new net: C80.1, C82.1, R128.1, U23.19 (VSTOR)
- new net: Q1.2 (S), R1.1, R2.2
- new net: R1.2, U1.7 (~{RESET})
- new net: C81.1, C83.1, L4.2, U23.14 (VOUT), U24.1 (VDD), U24.3 (EN)
- new net: C84.1, R133.2, U24.5 (OUT)
- new net: D10.1 (K), D11.2 (A), SC3.1 (V+), SC4.2 (V-)
- new net: D14.2 (A), R136.1
- new net: R122.1, R123.2, U23.10 (OK_HYST)
- new net: R127.1, R128.2, R130.2, U23.3 (VOC_SAMP)
- new net: U1.1 (~{MR}), U1.8 (~{WDO})
- new net: D6.1 (K), D9.2 (A), SC2.1 (V+)
- new net: D12.1 (K), D13.2 (A), SC5.1 (V+)
- new net: D11.1 (K), D12.2 (A), SC4.1 (V+), SC5.2 (V-)
- new net: R123.1, R124.2, U23.11 (OK_PROG)
- new net: C77.1, U23.4 (VREF_SAMP)
- new net: L4.1, U23.16 (LBUCK)
- new net: L3.2, U23.20 (LBOOST)
- new net: U12.3 (NC), U12.6 (NC)
- new net: D15.2 (A), R137.1
- new net BAT_P: R139.2
- new net I2C_LIGHT_SDA: U12.8 (SDA)
- new net VBAT_OK_BOTTOM: R129.1, U23.13 (VBAT_OK)
- new net VBAT_OK_TOP: R110.1, U16.13 (VBAT_OK)
- new net VLXSMPS: L5.1
- new net VOUT_EN_BOTTOM: C78.1, R129.2, R135.1, U23.6 (VOUT_EN)
- new net VSOLAR_BOTTOM: C75.1, C76.1, D13.1 (K), D7.1 (K), L3.1, R127.2, U23.2 (VIN_DC)
- new net VUSB: D15.1 (K)
- no-connect marks 3 -> 5
Other:
- note added: "Check datasheet for suggested capacitor"
- note added: "Check datasheet for suggested inductance"
- note added: "Datasheet: https://www.st.com/resource/en/datasheet/dm00768509.pdf (See pg. 179 for power supply instructions)"
- note added: "For LED I=0.1mA, V=1.7V"
- note added: "Light Sensor"
- note added: "Solar Power Bottom"
- note added: "Solar Power Top"
- note added: "Status LEDs"
- note added: "Voltage divider to reduce battery 4.2V to ~3V assuming 3μA consumption"
- note added: "WATCH-DOG TIMER"
- note added: "WDT able to reset MCU when WDT_EN is high"
- note removed: "Energy Harvesting IC"
- moved on the sheet: C45, C46, C48, C56, C57, C61, C62, C63, C64, C72, D2, D4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
