File: old_stuff.kicad_sch (KiCad schematic)
At the start: 239 parts, among them J1 Micro_SD_Card, J10 TFM-110-12-X-D-A, J11 FLE-107-01-X-DV-A, J12 USD-1040310811, J14 FTS-105-01-X-DV-A, J2 U.FL-R-SMT-1, J3 USB_C_Receptacle_USB2.0, J4 SFC-110-T2-X-D-A, J5 TFM-110-12-X-D-A, J6 USB_C_Receptacle_USB2.0, J7 02x05 M 1.27mm, J8 Conn_01x08, J9 Conn_01x08, Q1 IRLML2803, Q10 MBT2222ADW1T1, Q11 NX3008NBKS, Q12 NX3008NBKS, Q13 MBT2222ADW1T1, Q14 MBT2222ADW1T1, Q15 NX3008NBKS, Q16 NX3008NBKS, Q17 MBT2222ADW1T1, Q18 MBT2222ADW1T1, Q19 MMBT2907, Q2 SQ3495EV-T1, Q20 MMBT2907, Q21 SQ3495EV-T1, Q3 NX3008NBKS, Q4 NX3008NBKS, Q5 MBT2222ADW1T1, Q6 MBT2222ADW1T1, Q7 NX3008NBKS, Q8 NX3008NBKS, Q9 MBT2222ADW1T1, SW1 CAS-120TA, SW2 KMR2x, SW3 CAS-120TA, U1 MAX706RESA+, U10 BNO085, U11 USBLC6-2SC6, U12 STM32H743VITx, U13 WE-TVS-82400102, U14 OPT4001, U15 LTC4412xS6, U17 XC6210B332MR-G, U18 AP7366-28W5-7, U19 TLV75515PDBVR, U2 DRV8830DRC, U3 LTC4412xS6, U4 DRV8830DRC, U5 PCF8523TK, U6 DRV8830DRC, U7 AP2112K-3.3, U8 MR25H40, U9 RFM98PW, Y1 32.768kHz/7pF, Y2 32.768kHz/12.5pF, Y3 12MHz/7pF

Commit message: Complete MCU planning
Parts:
- removed C14, C15, C18, C19, C22, C23, C26, C27: 10nF, Capacitor_SMD:C_0603_1608Metric, symbol Device:C
- removed C2, C29, C30, C35, C37, C38, C39: 0.1uF, Capacitor_SMD:C_0603_1608Metric, symbol Device:C_Small
- removed C28: 47uF, Capacitor_Tantalum_SMD:CP_EIA-2012-12_Kemet-R, symbol Device:C_Polarized_Small_US
- removed C32, C36: 2.2uF, Capacitor_SMD:C_0603_1608Metric, symbol Device:C_Small
- removed C33, C34: 4pF, Capacitor_SMD:C_0603_1608Metric, symbol Device:C_Small
- removed C40: 10nF, Capacitor_SMD:C_0603_1608Metric, symbol Device:C_Small
- removed C41, C42: 1uF, Capacitor_SMD:C_0603_1608Metric, symbol Device:C_Small
- removed C43: 0.1uF, Capacitor_SMD:C_0402_1005Metric, symbol Device:C
- removed FB1: 120R, Inductor_SMD:L_0603_1608Metric, symbol Device:FerriteBead_Small
- removed Q1: IRLML2803, Package_TO_SOT_SMD:SOT-23, symbol Transistor_FET:IRLML2060
- removed Q10, Q13, Q14, Q17, Q18, Q5, Q6, Q9: MBT2222ADW1T1, Package_TO_SOT_SMD:SOT-363_SC-70-6, symbol Transistor_BJT:MBT2222ADW1T1
- removed Q11, Q12, Q15, Q16, Q3, Q4, Q7, Q8: NX3008NBKS, Package_TO_SOT_SMD:SOT-363_SC-70-6, symbol mainboard:NX3008NBKS
- removed Q19, Q20: MMBT2907, Package_TO_SOT_SMD:SOT-23, symbol mainboard:MMBT2907
- removed R1, R77, R78: 0R, Resistor_SMD:R_0603_1608Metric, symbol Device:R_US
- removed R13, R14, R25, R26, R38, R39, R63, R64: 680R, Resistor_SMD:R_0603_1608Metric, symbol Device:R_US
- removed R15, R16, R27, R28, R40, R41, R65, R66: 100K, Resistor_SMD:R_0603_1608Metric, symbol Device:R_US
- removed R17, R18, R19, R21, R29, R30, R33, R35, R56, R57, R59, R61, R69, R70, R71, R73: 10K, Resistor_SMD:R_0603_1608Metric, symbol Device:R_US
- removed R2, R44, R45, R46, R47, R48, R49, R50, R51, R67, R68: DNI (0R), Resistor_SMD:R_0603_1608Metric, symbol Device:R_US
- removed R20, R22, R3, R34, R36, R60, R62, R72, R74: 200K, Resistor_SMD:R_0603_1608Metric, symbol Device:R_US
- removed R76, R88, R89: 10K, Resistor_SMD:R_0603_1608Metric, symbol Device:R_Small
- removed R82, R83: 4.7K, Resistor_SMD:R_0603_1608Metric, symbol Device:R_US
- removed R84, R85, R86, R87: 1K, Resistor_SMD:R_0603_1608Metric, symbol Device:R_US
- removed R90, R91: 0R, Resistor_SMD:R_0402_1005Metric, symbol Device:R_Small_US
- removed U1: MAX706RESA+, Package_SO:SOIC-8_3.9x4.9mm_P1.27mm, symbol mainboard:MAX708RESA+
- removed U12: STM32H743VITx, Package_QFP:LQFP-100_14x14mm_P0.5mm, symbol MCU_ST_STM32H7:STM32H743VITx
- removed U14: OPT4001, Package_TO_SOT_SMD:SOT-583-8, symbol solarpanels:OPT4001
- removed Y3: 12MHz/7pF, Crystal:Crystal_SMD_2520-4Pin_2.5x2.0mm, symbol Device:Crystal_GND24_Small
- added C74: 0.1uF, Capacitor_SMD:C_0603_1608Metric, symbol Device:C_Small
- added J15: BM02B-SRSS-TB, Connector_JST:JST_SH_BM02B-SRSS-TB_1x02-1MP_P1.00mm_Vertical, symbol Connector_Generic:Conn_01x02
- added R119: 0.04R, batteryboard:R_2512_CurrentSense, symbol Device:R_Small
- added R138: 0, Resistor_SMD:R_0603_1608Metric, symbol Device:R_Small_US
- added SW4: D2F-L2-A1, solarpanels:D2F-L2-A1, symbol Switch:SW_SPDT
- added SW5: D2F-L2-A, solarpanels:D2F-L2-A, symbol Switch:SW_SPDT
- added U22: INA219BxD, Package_SO:SOIC-8_3.9x4.9mm_P1.27mm, symbol Sensor_Energy:INA219BxD
Connections:
- net +3V3: now also C74.1, U22.5 (VS)
- net BATT_N_SW: now also J15.1 (Pin_1), SW5.2 (B)
- net BATT_P: now also SW4.3 (C)
- net BATT_P_SW: now also J15.2 (Pin_2), R119.2, SW4.2 (B), U22.7 (IN-)
- net GND: now also C74.2, R138.2, U22.1 (A1), U22.2 (A0), U22.6 (GND)
- net UART3_RX renamed UART_MB_TX
- net UART3_TX renamed UART_MB_RX
- new net: R138.1, SW5.3 (C)
- new net BATT_P_SENSE: R119.1, U22.8 (IN+)
- new net SCL_C_SENSE: U22.4 (SCL)
- new net SDA_C_SENSE: U22.3 (SDA)
- no-connect marks 56 -> 29
Other:
- note added: "Battery Connector and Disengage"
- note added: "Battery Current Draw Sensor"
- note added: "Current Sense Resistor ~5W"
- note added: "I2C 1 Addr 0x40"
- note removed: "Bus Protection - Bypass Jumpers"
- note removed: "Check Xtal Datasheet This value assumes 7pF crystal bulk capacitance"
- note removed: "DNI"
- note removed: "ESR < 100 mOhm Tol < 20%"
- note removed: "I2C Bus Protection - Motor1"
- note removed: "I2C Bus Protection - Motor2"
- note removed: "I2C Bus Protection - Motor3"
- note removed: "I2C Bus Protection - RTC"
- note removed: "Light Sensor"
- note removed: "MCU (STM32H743VITx)"
- note removed: "Motor 1 Jumpers"
- note removed: "Motor 2 Jumpers"
- note removed: "Motor 3 Jumpers"
- note removed: "NOTE"
- note removed: "RTC Jumpers"
- note removed: "Radio Jumper"
- note removed: "SD Card Jumper"
- note removed: "SPI Bus Protection - Radio"
- note removed: "SPI Bus Protection - SD Card"
- note removed: "These novel bus protection circuits prevent traditional I2C/SPI failure modes where a single slave failure can disable the entire bus. Learn more: https://doi.org/10.36227/techrxiv.15166620 By default, slave clock and/or data lines can be held low and the Master (SAMD51) will still be able to communicate with the remainder of the bus. They can individually be bypassed by removing the transistor(s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"
- note removed: "WATCH-DOG TIMER"
- note removed: "WDT able to reset MCU when WDT_EN is high"

Commit message: Implement most components
Parts:
- removed C10, C12: 10uF, Capacitor_SMD:C_0805_2012Metric, symbol Device:C_Small
- removed C11, C16, C20, C21, C74: 0.1uF, Capacitor_SMD:C_0603_1608Metric, symbol Device:C_Small
- removed C13: 1uF, Capacitor_SMD:C_0805_2012Metric, symbol Device:C_Small
- removed C17, C31: 4.7nF, Capacitor_SMD:C_0603_1608Metric, symbol Device:C_Small
- removed C24, C25: 22pF, Capacitor_SMD:C_0603_1608Metric, symbol Device:C_Small
- removed C3, C5, C53, C54, C55, C58, C59, C60, C9: 1uF, Capacitor_SMD:C_0603_1608Metric, symbol Device:C_Small
- removed C50, C51, C52: 10uF, Capacitor_SMD:C_0603_1608Metric, symbol Device:C_Small
- removed D1: MBR1020VL-AU_R1, Diode_SMD:D_SOD-123F, symbol Device:D_Schottky_Small
- removed J1: Micro_SD_Card, mainboard:microSD_104031-0811, symbol Connector:Micro_SD_Card_Det2
- removed J15: BM02B-SRSS-TB, Connector_JST:JST_SH_BM02B-SRSS-TB_1x02-1MP_P1.00mm_Vertical, symbol Connector_Generic:Conn_01x02
- removed J2: U.FL-R-SMT-1, mainboard:U.FL-R-SMT-1, symbol mainboard:U.FL-R-SMT-1
- removed J3, J6: USB_C_Receptacle_USB2.0, Connector_USB:USB_C_Receptacle_HRO_TYPE-C-31-M-12, symbol Connector:USB_C_Receptacle_USB2.0
- removed Q2: SQ3495EV-T1, Package_TO_SOT_SMD:SOT-23-6, symbol cameraboard:SQ3495EV-T1
- removed R10, R11, R24, R42, R7, R8, R9: 10K, Resistor_SMD:R_0603_1608Metric, symbol Device:R_US
- removed R119: 0.04R, batteryboard:R_2512_CurrentSense, symbol Device:R_Small
- removed R138: 0, Resistor_SMD:R_0603_1608Metric, symbol Device:R_Small_US
- removed R23: 1M, Resistor_SMD:R_0603_1608Metric, symbol Device:R_US
- removed R31, R32: 5.1K, Resistor_SMD:R_0603_1608Metric, symbol Device:R_US
- removed R37, R58: 22R, Resistor_SMD:R_0603_1608Metric, symbol Device:R_US
- removed R43: 0R, Resistor_SMD:R_0603_1608Metric, symbol Device:R_US
- removed R52: 100K, Resistor_SMD:R_0603_1608Metric, symbol Device:R_US
- removed R75: 1M, Resistor_SMD:R_0603_1608Metric, symbol Device:R_Small
- removed R79: 0R, Resistor_SMD:R_0603_1608Metric, symbol Device:R_Small
- removed R80, R81: 5.1K, Resistor_SMD:R_0603_1608Metric, symbol Device:R_Small
- removed SW4: D2F-L2-A1, solarpanels:D2F-L2-A1, symbol Switch:SW_SPDT
- removed SW5: D2F-L2-A, solarpanels:D2F-L2-A, symbol Switch:SW_SPDT
- removed U10: BNO085, mainboard:BNO085, symbol mainboard:BNO085
- removed U11: USBLC6-2SC6, Package_TO_SOT_SMD:SOT-23-6, symbol Power_Protection:USBLC6-2SC6
- removed U13: WE-TVS-82400102, Package_TO_SOT_SMD:SOT-23-6, symbol Power_Protection:USBLC6-2SC6
- removed U17: XC6210B332MR-G, Package_TO_SOT_SMD:SOT-23-5, symbol Regulator_Linear:AP2127K-2.8
- removed U18: AP7366-28W5-7, Package_TO_SOT_SMD:SOT-23-5, symbol Regulator_Linear:AP2127K-2.8
- removed U19: TLV75515PDBVR, Package_TO_SOT_SMD:SOT-23-5, symbol Regulator_Linear:AP2127K-2.8
- removed U22: INA219BxD, Package_SO:SOIC-8_3.9x4.9mm_P1.27mm, symbol Sensor_Energy:INA219BxD
- removed U3: LTC4412xS6, Package_TO_SOT_SMD:TSOT-23-6, symbol Power_Management:LTC4412xS6
- removed U7: AP2112K-3.3, Package_TO_SOT_SMD:SOT-23-5, symbol Regulator_Linear:AP2112K-3.3
- removed U8: MR25H40, mainboard:MR25H40DF, symbol Memory_NVRAM:MR25H40
- removed U9: RFM98PW, mainboard:RFM98PW, symbol mainboard:RFM98PW
- removed Y2: 32.768kHz/12.5pF, Crystal:Crystal_SMD_MicroCrystal_CC7V-T1A-2Pin_3.2x1.5mm, symbol Device:Crystal_Small
Connections:
- no-connect marks 29 -> 12
Other:
- note removed: "Battery Connector and Disengage"
- note removed: "Battery Current Draw Sensor"
- note removed: "Current Sense Resistor ~5W"
- note removed: "Default HI_POW to USB power. Use battery power when USB absent."
- note removed: "FLASH STORAGE"
- note removed: "HI-POW SELECT"
- note removed: "High Power Line Source Selection"
- note removed: "I2C 1 Addr 0x40"
- note removed: "IMU"
- note removed: "IMU datasheet recommends 12.5pF crystal capacitance"
- note removed: "LDOs"
- note removed: "Potentially Replace with Ferrite Bead"
- note removed: "Power Capacitors (0805)"
- note removed: "REGULATOR"
- note removed: "SD Card"
- note removed: "Shield"
- note removed: "UHF RADIO"
- note removed: "USB CONN"
- note removed: "USB Connector"
- note removed: "USB ESD Protection"

Commit message: Remove unused old stuff
Parts:
- removed C44, C49, C68: 1uF, Capacitor_SMD:C_0603_1608Metric, symbol Device:C_Small
- removed C47: 0.1uF, Capacitor_SMD:C_0603_1608Metric, symbol Device:C_Small
- removed C66: 47uF, Capacitor_Tantalum_SMD:CP_EIA-2012-12_Kemet-R, symbol Device:C_Polarized_Small_US
- removed D3: MBR1020VL-AU_R1, Diode_SMD:D_SOD-123F, symbol Device:D_Schottky_Small
- removed H1, H2, H3, H4, H5, H6, H7, H8: MountingHole_Pad, mainboard:MountingHole, symbol Mechanical:MountingHole_Pad
- removed J12: USD-1040310811, Connector_Card:microSD_HC_Molex_104031-0811, symbol cameraboard:USD-1040310811
- removed J7: 02x05 M 1.27mm, Connector_PinHeader_1.27mm:PinHeader_2x05_P1.27mm_Vertical_SMD, symbol Connector_Generic:Conn_02x05_Odd_Even
- removed J8, J9: Conn_01x08, Connector_PinHeader_2.54mm:PinHeader_1x08_P2.54mm_Vertical, symbol Connector_Generic:Conn_01x08
- removed Q21: SQ3495EV-T1, Package_TO_SOT_SMD:SOT-23-6, symbol cameraboard:SQ3495EV-T1
- removed R102: 1K, Resistor_SMD:R_0603_1608Metric, symbol Device:R_Small
- removed R105, R113, R114, R115, R116, R117, R118, R95, R96: 10K, Resistor_SMD:R_0603_1608Metric, symbol Device:R_Small
- removed R92: 100R, Resistor_SMD:R_0603_1608Metric, symbol Device:R_Small
- removed SW1, SW3: CAS-120TA, cameraboard:CAS-120TA, symbol Switch:SW_SPDT
- removed SW2: KMR2x, mainboard:BTN_KMR2, symbol Switch:SW_Push
- removed TP1, TP2, TP3, TP4: TP, TestPoint:TestPoint_THTPad_D1.0mm_Drill0.5mm, symbol Connector:TestPoint
- removed U15: LTC4412xS6, Package_TO_SOT_SMD:TSOT-23-6, symbol Power_Management:LTC4412xS6
Connections:
- no-connect marks 12 -> 8
Other:
- note removed: "(Not Populated)"
- note removed: "Grounded Mounting Holes"
- note removed: "HI-Power Selection"
- note removed: "Mounting Holes"
- note removed: "Power Enable Circuit"
- note removed: "Reset & Boot0 Switches"
- note removed: "SD Card Connector"
- note removed: "SWD Connector"
- note removed: "Select boot mode Set "low" for normal operation. Set "high" for bootloader mode"
- note removed: "Set for flight"
- note removed: "Solar Panel Board +Y"
- note removed: "Status LED & IO headers"
- note removed: "Test Points"
- note removed: "Toggle LDO power on or controlled by Mainboard enable line (defaults to power off)"
- note removed: "cameraboard"
- note removed: "mainboard"
- moved on the sheet: C1, C4, C6, C7, C8, FL1, FL2, FL3, J10, J11, J14, J4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
